File: ESC_2016.sch (KiCad schematic (older format))
At the start: 11 parts

Commit message: asdf
Parts:
- added R? (x9): R, symbol R
Connections:
- net GND: now also R?.1, R?.1, R?.1
- new net: R?.1, R?.2, R?.2 (x3)
- new net: R?.2, R?.2, R?.2
- new net I_PHASE_A: R?.1
- new net I_PHASE_B: R?.1
- new net I_PHASE_C: R?.1
